File: BackPlane.brd (EAGLE design)
At the start: 134.6 x 116.5 mm, 1 part

Commit message: progress
Parts:
- added U$2, U$3, U$4: THICC_CONNECTOR, THICC_CONNECTOR:THICC_CONNECTOR
Connections:
- new net +12V: U$2.15, U$2.16, U$2.23, U$2.24, U$3.15, U$3.16, U$3.23, U$3.24, U$4.15, U$4.16, U$4.23, U$4.24
- new net +12V_GND: U$2.13, U$2.14, U$2.21, U$2.22, U$3.13, U$3.14, U$3.21, U$3.22, U$4.13, U$4.14, U$4.21, U$4.22
- new net +5V: U$2.11, U$2.12, U$2.19, U$2.20, U$3.11, U$3.12, U$3.19, U$3.20, U$4.11, U$4.12, U$4.19, U$4.20
- new net +5V_GND: U$2.10, U$2.17, U$2.18, U$2.9, U$3.10, U$3.17, U$3.18, U$3.9, U$4.10, U$4.17, U$4.18, U$4.9
- new net B1: U$2.P1-13, U$2.P1-14, U$2.P1-15, U$2.P1-16, U$2.P2-17, U$2.P2-18, U$2.P2-19, U$2.P2-20, U$4.P1-13, U$4.P1-14, U$4.P1-15, U$4.P1-16, U$4.P2-17, U$4.P2-18, U$4.P2-19, U$4.P2-20
- new net B2: U$2.P2-1, U$2.P2-2, U$2.P2-3, U$2.P2-4, U$2.P2-5, U$2.P2-6, U$2.P2-7, U$2.P2-8, U$4.P2-1, U$4.P2-2, U$4.P2-3, U$4.P2-4, U$4.P2-5, U$4.P2-6, U$4.P2-7, U$4.P2-8
- new net B3: U$2.P3-25, U$2.P3-26, U$2.P3-27, U$2.P3-28, U$2.P4-5, U$2.P4-6, U$2.P4-7, U$2.P4-8, U$3.P3-25, U$3.P3-26, U$3.P3-27, U$3.P3-28, U$3.P4-5, U$3.P4-6, U$3.P4-7, U$3.P4-8, U$4.P3-25, U$4.P3-26, U$4.P3-27, U$4.P3-28, U$4.P4-5, U$4.P4-6, U$4.P4-7, U$4.P4-8
- new net B4: U$2.P3-13, U$2.P3-14, U$2.P3-15, U$2.P3-16, U$2.P4-10, U$2.P4-11, U$2.P4-12, U$2.P4-9, U$3.P3-13, U$3.P3-14, U$3.P3-15, U$3.P3-16, U$3.P4-10, U$3.P4-11, U$3.P4-12, U$3.P4-9, U$4.P3-13, U$4.P3-14, U$4.P3-15, U$4.P3-16, U$4.P4-10, U$4.P4-11, U$4.P4-12, U$4.P4-9
- new net B5: U$3.P1-13, U$3.P1-14, U$3.P1-15, U$3.P1-16, U$3.P2-17, U$3.P2-18, U$3.P2-19, U$3.P2-20
- new net B6: U$3.P2-1, U$3.P2-2, U$3.P2-3, U$3.P2-4, U$3.P2-5, U$3.P2-6, U$3.P2-7, U$3.P2-8
- new net CAN_H: U$2.8, U$3.8, U$4.8
- new net CAN_L: U$2.7, U$3.7, U$4.7
- new net R1: U$2.P1-1, U$2.P1-2, U$2.P1-21, U$2.P1-22, U$2.P1-23, U$2.P1-24, U$2.P1-3, U$2.P1-4, U$4.P1-1, U$4.P1-2, U$4.P1-21, U$4.P1-22, U$4.P1-23, U$4.P1-24, U$4.P1-3, U$4.P1-4
- new net R2: U$2.P1-10, U$2.P1-11, U$2.P1-12, U$2.P1-9, U$2.P2-13, U$2.P2-14, U$2.P2-15, U$2.P2-16, U$4.P1-10, U$4.P1-11, U$4.P1-12, U$4.P1-9, U$4.P2-13, U$4.P2-14, U$4.P2-15, U$4.P2-16
- new net R3: U$2.P3-17, U$2.P3-18, U$2.P3-19, U$2.P3-20, U$2.P4-13, U$2.P4-14, U$2.P4-15, U$2.P4-16, U$3.P3-17, U$3.P3-18, U$3.P3-19, U$3.P3-20, U$4.P3-17, U$4.P3-18, U$4.P3-19, U$4.P3-20, U$4.P4-13, U$4.P4-14, U$4.P4-15, U$4.P4-16
- new net R4: U$2.P3-1, U$2.P3-2, U$2.P3-3, U$2.P3-4, U$2.P3-5, U$2.P3-6, U$2.P3-7, U$2.P3-8, U$3.P3-1, U$3.P3-2, U$3.P3-3, U$3.P3-4, U$3.P3-5, U$3.P3-6, U$3.P3-7, U$3.P3-8, U$4.P3-1, U$4.P3-2, U$4.P3-3, U$4.P3-4, U$4.P3-5, U$4.P3-6, U$4.P3-7, U$4.P3-8
- new net R5: U$3.P1-1, U$3.P1-2, U$3.P1-21, U$3.P1-22, U$3.P1-23, U$3.P1-24, U$3.P1-3, U$3.P1-4
- new net R6: U$3.P1-10, U$3.P1-11, U$3.P1-12, U$3.P1-9, U$3.P2-13, U$3.P2-14, U$3.P2-15, U$3.P2-16
- new net R7: U$3.P4-13, U$3.P4-14, U$3.P4-15, U$3.P4-16
- new net Y1: U$2.P1-17, U$2.P1-18, U$2.P1-19, U$2.P1-20, U$2.P2-21, U$2.P2-22, U$2.P2-23, U$2.P2-24, U$4.P1-17, U$4.P1-18, U$4.P1-19, U$4.P1-20, U$4.P2-21, U$4.P2-22, U$4.P2-23, U$4.P2-24
- new net Y2: U$2.P1-5, U$2.P1-6, U$2.P1-7, U$2.P1-8, U$2.P2-10, U$2.P2-11, U$2.P2-12, U$2.P2-9, U$4.P1-5, U$4.P1-6, U$4.P1-7, U$4.P1-8, U$4.P2-10, U$4.P2-11, U$4.P2-12, U$4.P2-9
- new net Y3: U$2.P4-17, U$2.P4-18, U$2.P4-19, U$2.P4-20, U$2.P4-25, U$2.P4-26, U$2.P4-27, U$2.P4-28, U$4.P4-17, U$4.P4-18, U$4.P4-19, U$4.P4-20, U$4.P4-25, U$4.P4-26, U$4.P4-27, U$4.P4-28
- new net Y4: U$2.P3-10, U$2.P3-11, U$2.P3-12, U$2.P3-9, U$2.P4-1, U$2.P4-2, U$2.P4-3, U$2.P4-4, U$3.P3-10, U$3.P3-11, U$3.P3-12, U$3.P3-9, U$3.P4-1, U$3.P4-2, U$3.P4-3, U$3.P4-4, U$4.P3-10, U$4.P3-11, U$4.P3-12, U$4.P3-9, U$4.P4-1, U$4.P4-2, U$4.P4-3, U$4.P4-4
- new net Y5: U$3.P1-17, U$3.P1-18, U$3.P1-19, U$3.P1-20, U$3.P2-21, U$3.P2-22, U$3.P2-23, U$3.P2-24
- new net Y6: U$3.P1-5, U$3.P1-6, U$3.P1-7, U$3.P1-8, U$3.P2-10, U$3.P2-11, U$3.P2-12, U$3.P2-9
- new net Y7: U$3.P4-17, U$3.P4-18, U$3.P4-19, U$3.P4-20, U$3.P4-25, U$3.P4-26, U$3.P4-27, U$3.P4-28

Commit message: names
Connections:
- new net B10: U$4.P2-1, U$4.P2-2, U$4.P2-3, U$4.P2-4, U$4.P2-5, U$4.P2-6, U$4.P2-7, U$4.P2-8
- new net B11: U$4.P3-25, U$4.P3-26, U$4.P3-27, U$4.P3-28, U$4.P4-5, U$4.P4-6, U$4.P4-7, U$4.P4-8
- new net B12: U$4.P3-13, U$4.P3-14, U$4.P3-15, U$4.P3-16, U$4.P4-10, U$4.P4-11, U$4.P4-12, U$4.P4-9
- new net B7: U$3.P4-5, U$3.P4-6, U$3.P4-7, U$3.P4-8
- new net B8: U$3.P3-13, U$3.P3-14, U$3.P3-15, U$3.P3-16, U$3.P4-10, U$3.P4-11, U$3.P4-12, U$3.P4-9
- new net B9: U$4.P1-13, U$4.P1-14, U$4.P1-15, U$4.P1-16, U$4.P2-17, U$4.P2-18, U$4.P2-19, U$4.P2-20
- new net BY: U$3.P3-25, U$3.P3-26, U$3.P3-27, U$3.P3-28
- new net R10: U$4.P1-10, U$4.P1-11, U$4.P1-12, U$4.P1-9, U$4.P2-13, U$4.P2-14, U$4.P2-15, U$4.P2-16
- new net R11: U$4.P3-17, U$4.P3-18, U$4.P3-19, U$4.P3-20, U$4.P4-13, U$4.P4-14, U$4.P4-15, U$4.P4-16
- new net R12: U$4.P3-1, U$4.P3-2, U$4.P3-3, U$4.P3-4, U$4.P3-5, U$4.P3-6, U$4.P3-7, U$4.P3-8
- new net R8: U$3.P3-1, U$3.P3-2, U$3.P3-3, U$3.P3-4, U$3.P3-5, U$3.P3-6, U$3.P3-7, U$3.P3-8
- new net R9: U$4.P1-1, U$4.P1-2, U$4.P1-21, U$4.P1-22, U$4.P1-23, U$4.P1-24, U$4.P1-3, U$4.P1-4
- new net Y10: U$4.P1-5, U$4.P1-6, U$4.P1-7, U$4.P1-8, U$4.P2-10, U$4.P2-11, U$4.P2-12, U$4.P2-9
- new net Y11: U$4.P4-17, U$4.P4-18, U$4.P4-19, U$4.P4-20, U$4.P4-25, U$4.P4-26, U$4.P4-27, U$4.P4-28
- new net Y12: U$4.P3-10, U$4.P3-11, U$4.P3-12, U$4.P3-9, U$4.P4-1, U$4.P4-2, U$4.P4-3, U$4.P4-4
- new net Y8: U$3.P3-10, U$3.P3-11, U$3.P3-12, U$3.P3-9, U$3.P4-1, U$3.P4-2, U$3.P4-3, U$3.P4-4
- new net Y9: U$4.P1-17, U$4.P1-18, U$4.P1-19, U$4.P1-20, U$4.P2-21, U$4.P2-22, U$4.P2-23, U$4.P2-24
- net B1: no longer U$4.P1-13, U$4.P1-14, U$4.P1-15, U$4.P1-16, U$4.P2-17, U$4.P2-18, U$4.P2-19, U$4.P2-20
- net B2: no longer U$4.P2-1, U$4.P2-2, U$4.P2-3, U$4.P2-4, U$4.P2-5, U$4.P2-6, U$4.P2-7, U$4.P2-8
- net B3: no longer U$3.P3-25, U$3.P3-26, U$3.P3-27, U$3.P3-28, U$3.P4-5, U$3.P4-6, U$3.P4-7, U$3.P4-8, U$4.P3-25, U$4.P3-26, U$4.P3-27, U$4.P3-28, U$4.P4-5, U$4.P4-6, U$4.P4-7, U$4.P4-8
- net B4: no longer U$3.P3-13, U$3.P3-14, U$3.P3-15, U$3.P3-16, U$3.P4-10, U$3.P4-11, U$3.P4-12, U$3.P4-9, U$4.P3-13, U$4.P3-14, U$4.P3-15, U$4.P3-16, U$4.P4-10, U$4.P4-11, U$4.P4-12, U$4.P4-9
- net R1: no longer U$4.P1-1, U$4.P1-2, U$4.P1-21, U$4.P1-22, U$4.P1-23, U$4.P1-24, U$4.P1-3, U$4.P1-4
- net R2: no longer U$4.P1-10, U$4.P1-11, U$4.P1-12, U$4.P1-9, U$4.P2-13, U$4.P2-14, U$4.P2-15, U$4.P2-16
- net R3: no longer U$3.P3-17, U$3.P3-18, U$3.P3-19, U$3.P3-20, U$4.P3-17, U$4.P3-18, U$4.P3-19, U$4.P3-20, U$4.P4-13, U$4.P4-14, U$4.P4-15, U$4.P4-16
- net R4: no longer U$3.P3-1, U$3.P3-2, U$3.P3-3, U$3.P3-4, U$3.P3-5, U$3.P3-6, U$3.P3-7, U$3.P3-8, U$4.P3-1, U$4.P3-2, U$4.P3-3, U$4.P3-4, U$4.P3-5, U$4.P3-6, U$4.P3-7, U$4.P3-8
- net R7: now also U$3.P3-17, U$3.P3-18, U$3.P3-19, U$3.P3-20
- net Y1: no longer U$4.P1-17, U$4.P1-18, U$4.P1-19, U$4.P1-20, U$4.P2-21, U$4.P2-22, U$4.P2-23, U$4.P2-24
- net Y2: no longer U$4.P1-5, U$4.P1-6, U$4.P1-7, U$4.P1-8, U$4.P2-10, U$4.P2-11, U$4.P2-12, U$4.P2-9
- net Y3: no longer U$4.P4-17, U$4.P4-18, U$4.P4-19, U$4.P4-20, U$4.P4-25, U$4.P4-26, U$4.P4-27, U$4.P4-28
- net Y4: no longer U$3.P3-10, U$3.P3-11, U$3.P3-12, U$3.P3-9, U$3.P4-1, U$3.P4-2, U$3.P4-3, U$3.P4-4, U$4.P3-10, U$4.P3-11, U$4.P3-12, U$4.P3-9, U$4.P4-1, U$4.P4-2, U$4.P4-3, U$4.P4-4

Commit message: Routing
Parts:
- moved U$3 122.5 mm to (64.8, 95.5)
- moved U$4 112.7 mm to (94.0, 53.4), turned to 240 degrees
Connections:
- removed net BY: U$3.P3-25, U$3.P3-26, U$3.P3-27, U$3.P3-28
- net +12V: now also U$2.7, U$2.8, U$3.7, U$3.8, U$4.7, U$4.8; no longer U$2.23, U$2.24, U$3.23, U$3.24, U$4.23, U$4.24
- net B7: now also U$3.P3-25, U$3.P3-26, U$3.P3-27, U$3.P3-28
- net CAN_H: now also U$2.24, U$3.24, U$4.24; no longer U$2.8, U$3.8, U$4.8
- net CAN_L: now also U$2.23, U$3.23, U$4.23; no longer U$2.7, U$3.7, U$4.7
Routing:
- added copper zone on layer 1, net B1
- added copper zone on layer 1, net B10
- added copper zone on layer 1, net B11
- added copper zone on layer 1, net B12
- added copper zone on layer 1, net B2
- added copper zone on layer 1, net B3
- added copper zone on layer 1, net B4
- added copper zone on layer 1, net B5
- added copper zone on layer 1, net B6
- added copper zone on layer 1, net B7
- added copper zone on layer 1, net B8
- added copper zone on layer 1, net B9
- added copper zone on layer 1, net R1
- added copper zone on layer 1, net R10
- added copper zone on layer 1, net R11
- added copper zone on layer 1, net R12
- added copper zone on layer 1, net R2
- added copper zone on layer 1, net R3
- added copper zone on layer 1, net R4
- added copper zone on layer 1, net R5
- added copper zone on layer 1, net R6
- added copper zone on layer 1, net R7
- added copper zone on layer 1, net R8
- added copper zone on layer 1, net R9
- added copper zone on layer 1, net Y1
- added copper zone on layer 1, net Y10
- added copper zone on layer 1, net Y11
- added copper zone on layer 1, net Y12
- added copper zone on layer 1, net Y2
- added copper zone on layer 1, net Y3
- added copper zone on layer 1, net Y4
- added copper zone on layer 1, net Y5
- added copper zone on layer 1, net Y6
- added copper zone on layer 1, net Y7
- added copper zone on layer 1, net Y8
- added copper zone on layer 1, net Y9

Commit message: connectors
Parts:
- added ESC5_CON1: 3PINCONNECTOR, afro_20A_esc:3PINCONNECTOR
Changed lines of the file:
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@@
 <layer number="48" name="Document" color="7" fill="1" visible="yes" active="yes"/>
 <layer number="49" name="Reference" color="7" fill="1" visible="yes" active="yes"/>
+<layer number="50" name="dxf" color="7" fill="1" visible="no" active="no"/>
 <layer number="51" name="tDocu" color="7" fill="1" visible="yes" active="yes"/>
 <layer number="52" name="bDocu" color="7" fill="1" visible="yes" active="yes"/>
+<layer number="53" name="tGND_GNDA" color="7" fill="9" visible="no" active="no"/>
+<layer number="54" name="bGND_GNDA" color="1" fill="9" visible="no" active="no"/>
+<layer number="56" name="wert" color="7" fill="1" visible="no" active="no"/>
+<layer number="57" name="tCAD" color="7" fill="1" visible="no" active="no"/>
+<layer number="59" name="tCarbon" color="7" fill="1" visible="no" active="no"/>
+<layer number="60" name="bCarbon" color="7" fill="1" visible="no" active="no"/>
 <layer number="88" name="SimResults" color="9" fill="1" visible="no" active="no"/>
 <layer number="89" name="SimProbes" color="9" fill="1" visible="no" active="no"/>
@@
 <layer number="97" name="Info" color="7" fill="1" visible="no" active="no"/>
 <layer number="98" name="Guide" color="6" fill="1" visible="no" active="no"/>
+<layer number="99" name="SpiceOrder" color="7" fill="1" visible="no" active="no"/>
+<layer number="100" name="Muster" color="7" fill="1" visible="no" active="no"/>
+<layer number="101" name="Patch_Top" color="12" fill="4" visible="yes" active="yes"/>
+<layer number="102" name="Vscore" color="7" fill="1" visible="yes" active="yes"/>
+<layer number="103" name="tMap" color="7" fill="1" visible="yes" active="yes"/>
+<layer number="104" name="Name" color="16" fill="1" visible="yes" active="yes"/>
+<layer number="105" name="tPlate" color="7" fill="1" visible="yes" active="yes"/>
+<layer number="106" name="bPlate" color="7" fill="1" visible="yes" active="yes"/>
+<layer number="107" name="Crop" color="7" fill="1" visible="yes" active="yes"/>
+<layer number="108" name="tplace-old" color="10" fill="1" visible="yes" active="yes"/>
+<layer number="109" name="ref-old" color="11" fill="1" visible="yes" active="yes"/>
+<layer number="110" name="fp0" color="7" fill="1" visible="yes" active="yes"/>
+<layer number="111" name="LPC17xx" color="7" fill="1" visible="yes" active="yes"/>
+<layer number="112" name="tSilk" color="7" fill="1" visible="yes" active="yes"/>
+<layer number="113" name="IDFDebug" color="4" fill="1" visible="yes" active="yes"/>
+<layer number="114" name="Badge_Outline" color="7" fill="1" visible="no" active="yes"/>
+<layer number="115" name="ReferenceISLANDS" color="7" fill="1" visible="no" active="yes"/>
+<layer number="116" name="Patch_BOT" color="9" fill="4" visible="yes" active="yes"/>
+<layer number="118" name="Rect_Pads" color="7" fill="1" visible="no" active="yes"/>
+<layer number="121" name="_tsilk" color="7" fill="1" visible="yes" active="yes"/>
+<layer number="122" name="_bsilk" color="7" fill="1" visible="yes" active="yes"/>
+<layer number="123" name="tTestmark" color="7" fill="1" visible="yes" active="yes"/>
+<layer number="124" name="bTestmark" color="7" fill="1" visible="yes" active="yes"/>
+<layer number="125" name="_tNames" color="7" fill="1" visible="yes" active="yes"/>
+<layer number="126" name="_bNames" color="7" fill="1" visible="yes" active="yes"/>
+<layer number="127" name="_tValues" color="7" fill="1" visible="yes" active="yes"/>
+<layer number="128" name="_bValues" color="7" fill="1" visible="yes" active="yes"/>
+<layer number="129" name="Mask" color="7" fill="1" visible="yes" active="yes"/>
+<layer number="131" name="tAdjust" color="7" fill="1" visible="yes" active="yes"/>
+<layer number="132" name="bAdjust" color="7" fill="1" visible="yes" active="yes"/>
+<layer number="144" name="Drill_legend" color="7" fill="1" visible="yes" active="yes"/>
+<layer number="150" name="Notes" color="7" fill="1" visible="yes" active="yes"/>
+<layer number="151" name="HeatSink" color="7" fill="1" visible="yes" active="yes"/>
+<layer number="152" name="_bDocu" color="7" fill="1" visible="yes" active="yes"/>
+<layer number="153" name="FabDoc1" color="7" fill="1" visible="yes" active="yes"/>
+<layer number="154" name="FabDoc2" color="7" fill="1" visible="yes" active="yes"/>
+<layer number="155" name="FabDoc3" color="7" fill="1" visible="yes" active="yes"/>
+<layer number="199" name="Contour" color="7" fill="1" visible="yes" active="yes"/>
+<layer number="200" name="200bmp" color="1" fill="10" visible="yes" active="yes"/>
+<layer number="201" name="201bmp" color="2" fill="10" visible="yes" active="yes"/>
+<layer number="202" name="202bmp" color="3" fill="10" visible="yes" active="yes"/>
+<layer number="203" name="203bmp" color="4" fill="10" visible="yes" active="yes"/>
+<layer number="204" name="204bmp" color="5" fill="10" visible="yes" active="yes"/>
+<layer number="205" name="205bmp" color="6" fill="10" visible="yes" active="yes"/>
+<layer number="206" name="206bmp" color="7" fill="10" visible="yes" active="yes"/>
+<layer number="207" name="207bmp" color="8" fill="10" visible="yes" active="yes"/>
+<layer number="208" name="208bmp" color="9" fill="10" visible="yes" active="yes"/>
+<layer number="209" name="209bmp" color="7" fill="1" visible="yes" active="yes"/>
+<layer number="210" name="210bmp" color="7" fill="1" visible="yes" active="yes"/>
+<layer number="211" name="211bmp" color="7" fill="1" visible="yes" active="yes"/>
+<layer number="212" name="212bmp" color="7" fill="1" visible="yes" active="yes"/>
+<layer number="213" name="213bmp" color="7" fill="1" visible="yes" active="yes"/>
+<layer number="214" name="214bmp" color="7" fill="1" visible="yes" active="yes"/>
+<layer number="215" name="215bmp" color="7" fill="1" visible="yes" active="yes"/>
+<layer number="216" name="216bmp" color="7" fill="1" visible="yes" active="yes"/>
+<layer number="217" name="217bmp" color="18" fill="1" visible="no" active="no"/>
+<layer number="218" name="218bmp" color="19" fill="1" visible="no" active="no"/>
+<layer number="219" name="219bmp" color="20" fill="1" visible="no" active="no"/>
+<layer number="220" name="220bmp" color="21" fill="1" visible="no" active="no"/>
+<layer number="221" name="221bmp" color="22" fill="1" visible="no" active="no"/>
+<layer number="222" name="222bmp" color="23" fill="1" visible="no" active="no"/>
+<layer number="223" name="223bmp" color="24" fill="1" visible="no" active="no"/>
+<layer number="224" name="224bmp" color="25" fill="1" visible="no" active="no"/>
+<layer number="225" name="225bmp" color="7" fill="1" visible="yes" active="yes"/>
+<layer number="226" name="226bmp" color="7" fill="1" visible="yes" active="yes"/>
+<layer number="227" name="227bmp" color="7" fill="1" visible="yes" active="yes"/>
+<layer number="228" name="228bmp" color="7" fill="1" visible="yes" active="yes"/>
+<layer number="229" name="229bmp" color="7" fill="1" visible="yes" active="yes"/>
+<layer number="230" name="230bmp" color="7" fill="1" visible="yes" active="yes"/>
+<layer number="231" name="231bmp" color="7" fill="1" visible="yes" active="yes"/>
+<layer number="232" name="Eagle3D_PG2" color="7" fill="1" visible="yes" active="yes"/>
+<layer number="233" name="Eagle3D_PG3" color="7" fill="1" visible="yes" active="yes"/>
+<layer number="248" name="Housing" color="7" fill="1" visible="yes" active="yes"/>
+<layer number="249" name="Edge" color="7" fill="1" visible="yes" active="yes"/>
+<layer number="250" name="Descript" color="3" fill="1" visible="no" active="no"/>
+<layer number="251" name="SMDround" color="12" fill="11" visible="no" active="no"/>
+<layer number="254" name="cooling" color="7" fill="1" visible="yes" active="yes"/>
+<layer number="255" name="routoute" color="7" fill="1" visible="yes" active="yes"/>
 </layers>
 <board>
@@
 <element name="U$3" library="THICC_CONNECTOR" package="THICC_CONNECTOR" value="THICC_CONNECTOR" x="64.8" y="95.45"/>
 <element name="U$4" library="THICC_CONNECTOR" package="THICC_CONNECTOR" value="THICC_CONNECTOR" x="94.05" y="53.4" rot="R240"/>
+<element name="ESC5_CON1" library="afro_20A_esc" package="3PINCONNECTOR" value="3PINCONNECTOR" x="-3.3" y="72" rot="R120">
+<attribute name="NAME" x="-3.056921875" y="61.978971875" size="1.27" layer="21" rot="R120"/>
+</element>
 </elements>
 <signals>

Commit message: routing
Parts:
- added ESC5_CON10, ESC5_CON11, ESC5_CON12, ESC5_CON2, ESC5_CON3, ESC5_CON4, ESC5_CON5, ESC5_CON6, ESC5_CON7, ESC5_CON8, ESC5_CON9: 3PINCONNECTOR, afro_20A_esc:3PINCONNECTOR
- moved ESC5_CON1 40.2 mm to (36.5, 78.0), flipped to the bottom, turned to 240 degrees
Connections:
- net B1: now also ESC5_CON1.C
- net B10: now also ESC5_CON10.C
- net B11: now also ESC5_CON11.C
- net B12: now also ESC5_CON12.C
- net B2: now also ESC5_CON2.C
- net B3: now also ESC5_CON3.C
- net B4: now also ESC5_CON4.C
- net B5: now also ESC5_CON5.C
- net B6: now also ESC5_CON6.C
- net B7: now also ESC5_CON7.C
- net B8: now also ESC5_CON8.C
- net B9: now also ESC5_CON9.C
- net R1: now also ESC5_CON1.A
- net R10: now also ESC5_CON10.A
- net R11: now also ESC5_CON11.A
- net R12: now also ESC5_CON12.A
- net R2: now also ESC5_CON2.A
- net R3: now also ESC5_CON3.A
- net R4: now also ESC5_CON4.A
- net R5: now also ESC5_CON5.A
- net R6: now also ESC5_CON6.A
- net R7: now also ESC5_CON7.A
- net R8: now also ESC5_CON8.A
- net R9: now also ESC5_CON9.A
- net Y1: now also ESC5_CON1.B
- net Y10: now also ESC5_CON10.B
- net Y11: now also ESC5_CON11.B
- net Y12: now also ESC5_CON12.B
- net Y2: now also ESC5_CON2.B
- net Y3: now also ESC5_CON3.B
- net Y4: now also ESC5_CON4.B
- net Y5: now also ESC5_CON5.B
- net Y6: now also ESC5_CON6.B
- net Y7: now also ESC5_CON7.B
- net Y8: now also ESC5_CON8.B
- net Y9: now also ESC5_CON9.B
Routing:
- added copper zone on layer 1, net +12V
- added copper zone on layer 1, net +12V_GND
- added copper zone on layer 1, net +5V
- added copper zone on layer 1, net +5V_GND

Commit message: routing
Parts:
- moved ESC5_CON12 332.7 mm to (106.6, 76.6), flipped to the bottom, turned to 120 degrees
- moved ESC5_CON11 291.6 mm to (97.8, 61.4), flipped to the bottom, turned to 120 degrees
- moved ESC5_CON10 245.8 mm to (86.7, 41.9), flipped to the bottom, turned to 120 degrees
- moved ESC5_CON8 241.7 mm to (56.0, 95.1), flipped to the bottom
- moved ESC5_CON7 214.5 mm to (38.4, 95.1), flipped to the bottom
- moved ESC5_CON9 204.7 mm to (77.9, 26.6), flipped to the bottom, turned to 120 degrees
- moved ESC5_CON6 198.8 mm to (78.5, 95.1), flipped to the bottom
- moved ESC5_CON5 182.5 mm to (96.1, 95.1), flipped to the bottom
- moved ESC5_CON4 91.2 mm to (48.0, 41.8), flipped to the bottom, turned to 240 degrees
- moved ESC5_CON3 61.6 mm to (56.8, 26.6), flipped to the bottom, turned to 240 degrees
- moved ESC5_CON2 8.52 mm to (37.0, 61.2)
- moved ESC5_CON1 8.45 mm to (28.1, 76.4)

Commit message: Update BackPlane.brd
Parts:
- moved ESC5_CON6 10.5 mm to (88.9, 96.2)
- moved ESC5_CON5 10.4 mm to (106.4, 96.2)
- moved ESC5_CON1 9.73 mm to (21.9, 83.9)
- moved ESC5_CON2 9.51 mm to (30.9, 68.5)
- moved ESC5_CON10 9.47 mm to (83.2, 33.1)
- moved ESC5_CON9 9.38 mm to (74.4, 17.9)
- moved ESC5_CON7 7.58 mm to (30.9, 96.2)
- moved ESC5_CON8 7.58 mm to (48.5, 96.2)
- moved ESC5_CON12 7.57 mm to (111.7, 82.2)
- moved ESC5_CON4 7.53 mm to (50.5, 34.7)
- moved ESC5_CON11 7.50 mm to (102.9, 66.9)
- moved ESC5_CON3 7.49 mm to (59.2, 19.5)

Commit message: Update BackPlane.brd
Parts:
- moved ESC5_CON11 18.0 mm to (112.2, 82.3)
- moved ESC5_CON12 17.2 mm to (103.4, 67.1)
- moved ESC5_CON2 1.03 mm to (30.2, 69.3)
- moved ESC5_CON4 1.00 mm to (50.7, 33.7)
- moved ESC5_CON10 1.00 mm to (83.2, 32.1)
- moved ESC5_CON9 1.00 mm to (74.4, 16.9)
- moved ESC5_CON1 0.88 mm to (21.4, 84.5)
- moved ESC5_CON3 0.88 mm to (59.4, 18.6)
- moved ESC5_CON8 0.56 mm to (48.0, 96.5)
- moved ESC5_CON7 0.50 mm to (30.5, 96.5)
Routing:
- net R1: track 0.00 -> 7.43 mm
- net Y1: track 0.00 -> 7.09 mm
- net R5: track 0.00 -> 6.79 mm
- net R6: track 0.00 -> 6.61 mm
- net B1: track 0.00 -> 6.56 mm
- net Y5: track 0.00 -> 6.52 mm
- net B10: track 0.00 -> 6.49 mm
- net B5: track 0.00 -> 6.45 mm
- net B9: track 0.00 -> 6.45 mm
- net Y10: track 0.00 -> 6.43 mm
- net Y7: track 0.00 -> 6.38 mm
- net B12: track 0.00 -> 6.33 mm
- net Y6: track 0.00 -> 6.29 mm
- net B6: track 0.00 -> 6.25 mm
- net R8: track 0.00 -> 6.23 mm
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