File: BackPlane.brd (EAGLE design)
At the start: 134.6 x 116.5 mm, 26 parts

Commit message: final stuff
Routing:
- net +12V_GND: track 77.6 -> 100.2 mm, vias 0 -> 3
- net +12V: track 76.8 -> 87.8 mm, vias 0 -> 3
- net CAN_L: track 285.8 -> 287.6 mm, vias 0 -> 1
- net CAN_H: track 299.8 -> 301.4 mm, vias 0 -> 1
- net +5V_GND: vias 1 -> 4
- net +5V: vias 0 -> 3
Changed lines of the file:
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@@
 <text x="12.301315625" y="101.0446" size="1.016" layer="25" rot="R240">5/64" Hex</text>
 <text x="32.2834" y="90.3986" size="1.016" layer="25">3/32" Hex</text>
-<text x="56.8452" y="81.8896" size="1.016" layer="25" rot="R90">+12V</text>
-<text x="71.5518" y="91.5162" size="1.016" layer="25" rot="R90">+12V_GND</text>
+<text x="55.9054" y="86.5124" size="1.016" layer="25" rot="R90">+12V</text>
+<text x="71.1962" y="84.9884" size="1.016" layer="25" rot="R90">+12V_GND</text>
 <text x="57.023" y="65.6336" size="1.016" layer="25" rot="R90">+12V</text>
 <text x="57.1246" y="45.9994" size="1.016" layer="25" rot="R90">+12V</text>
@@
 Jason King
 Tyler Stagge</text>
+<text x="52.7558" y="80.01" size="0.8128" layer="25">+5V</text>
+<text x="51.3588" y="68.2244" size="0.8128" layer="25">+12V</text>
+<text x="70.4342" y="99.6696" size="0.8128" layer="25">+5V</text>
+<text x="74.3204" y="94.3102" size="0.8128" layer="25">+5V_GND</text>
 </plain>
 <attributes>
@@
 <wire x1="25.757221875" y1="43.020415625" x2="34.00970625" y2="40.008084375" width="0.254" layer="1"/>
 <wire x1="69.8" y1="112.4" x2="73.025" y2="115.316" width="0.254" layer="16"/>
-<wire x1="73.025" y1="115.316" x2="113.538" y2="115.316" width="0.254" layer="16"/>
+<wire x1="73.025" y1="115.316" x2="80.645" y2="115.316" width="0.254" layer="16"/>
+<wire x1="80.645" y1="115.316" x2="113.538" y2="115.316" width="0.254" layer="16"/>
 <wire x1="113.538" y1="115.316" x2="133.223" y2="81.407" width="0.254" layer="16"/>
 <wire x1="133.223" y1="81.407" x2="114.935" y2="49.911" width="0.254" layer="16"/>
@@
 <wire x1="47.879" y1="1.651" x2="25.019" y2="41.529" width="0.254" layer="16"/>
 <wire x1="25.019" y1="41.529" x2="25.757221875" y2="43.020415625" width="0.254" layer="16"/>
+<via x="80.5942" y="113.5126" extent="1-16" drill="0.85"/>
+<wire x1="80.5942" y1="113.5126" x2="80.5942" y2="115.2652" width="0.254" layer="16"/>
+<wire x1="80.5942" y1="115.2652" x2="80.645" y2="115.316" width="0.254" layer="16"/>
 </signal>
 <signal name="CAN_H">
@@
 <wire x1="25.08181875" y1="40.348975" x2="47.625" y2="1.27" width="0.254" layer="1"/>
 <wire x1="47.625" y1="1.27" x2="86.868" y2="1.27" width="0.254" layer="1"/>
-<wire x1="20.955" y1="115.316" x2="65.024" y2="115.189" width="0.254" layer="1"/>
+<wire x1="20.955" y1="115.316" x2="54.559140625" y2="115.219159375" width="0.254" layer="1"/>
+<wire x1="54.559140625" y1="115.219159375" x2="65.024" y2="115.189" width="0.254" layer="1"/>
 <wire x1="65.024" y1="115.189" x2="67.8" y2="112.4" width="0.254" layer="1"/>
 <wire x1="112.014" y1="44.704" x2="86.868" y2="1.27" width="0.254" layer="1"/>
 <wire x1="107.681753125" y1="52.3308875" x2="112.014" y2="44.704" width="0.254" layer="1"/>
 <wire x1="26.757221875" y1="41.288365625" x2="25.08181875" y2="40.348975" width="0.254" layer="1"/>
+<via x="54.5846" y="113.665" extent="1-16" drill="0.85"/>
+<wire x1="54.5846" y1="113.665" x2="54.5846" y2="115.1937" width="0.254" layer="1"/>
+<wire x1="54.5846" y1="115.1937" x2="54.559140625" y2="115.219159375" width="0.254" layer="1"/>
 </signal>
 <signal name="+12V">
@@
 <wire x1="54.013196875" y1="56.426196875" x2="60.324121875" y2="56.426196875" width="2.54" layer="16"/>
 <wire x1="52.451" y1="54.864" x2="54.013196875" y2="56.426196875" width="2.54" layer="16"/>
+<via x="50.3428" y="70.2564" extent="1-16" drill="0.85"/>
+<via x="52.5018" y="70.2564" extent="1-16" drill="0.85"/>
+<via x="54.61" y="70.231" extent="1-16" drill="0.85"/>
+<wire x1="50.3428" y1="70.2564" x2="52.5018" y2="70.2564" width="1.016" layer="1"/>
+<wire x1="54.61" y1="70.231" x2="54.5846" y2="70.2564" width="1.016" layer="1"/>
+<wire x1="54.5846" y1="70.2564" x2="52.5018" y2="70.2564" width="1.016" layer="1"/>
+<wire x1="54.61" y1="70.231" x2="57.382109375" y2="73.003109375" width="1.016" layer="1"/>
+<wire x1="57.382109375" y1="73.003109375" x2="60.254415625" y2="73.003109375" width="1.016" layer="1"/>
 </signal>
 <signal name="+12V_GND">
@@
 <wire x1="51.562" y1="66.167" x2="67.31" y2="66.167" width="2.54" layer="16"/>
 <wire x1="46.99" y1="61.595" x2="51.562" y2="66.167" width="2.54" layer="16"/>
+<via x="50.3428" y="72.7456" extent="1-16" drill="0.85"/>
+<via x="52.5018" y="72.7202" extent="1-16" drill="0.85"/>
+<via x="54.6862" y="72.644" extent="1-16" drill="0.85"/>
+<wire x1="54.6862" y1="72.644" x2="54.61" y2="72.7202" width="1.016" layer="16"/>
+<wire x1="54.61" y1="72.7202" x2="52.5018" y2="72.7202" width="1.016" layer="16"/>
+<wire x1="50.3428" y1="72.7456" x2="50.3682" y2="72.7202" width="1.016" layer="16"/>
+<wire x1="50.3682" y1="72.7202" x2="52.5018" y2="72.7202" width="1.016" layer="16"/>
+<wire x1="54.6862" y1="72.644" x2="54.6862" y2="76.6318" width="1.016" layer="16"/>
+<wire x1="54.6862" y1="76.6318" x2="56.6928" y2="78.6384" width="1.016" layer="16"/>
+<wire x1="56.6928" y1="78.6384" x2="62.992" y2="78.6384" width="1.016" layer="16"/>
+<wire x1="64.680884375" y1="76.949515625" x2="67.37858125" y2="76.949515625" width="1.016" layer="16"/>
+<wire x1="62.992" y1="78.6384" x2="64.680884375" y2="76.949515625" width="1.016" layer="16"/>
 </signal>
 <signal name="+5V">
@@
 <wire x1="49.022" y1="80.645" x2="49.911" y2="81.534" width="2.54" layer="16"/>
 <wire x1="49.911" y1="81.534" x2="54.864" y2="81.534" width="2.54" layer="16"/>
+<via x="71.501" y="98.7298" extent="1-16" drill="0.85"/>
+<via x="71.5772" y="94.1832" extent="1-16" drill="0.85"/>
+<via x="71.5264" y="96.393" extent="1-16" drill="0.85"/>
 </signal>
 <signal name="+5V_GND">
@@
 <wire x1="36.576" y1="59.309" x2="39.497" y2="57.404" width="2.54" layer="1"/>
 <wire x1="30.789115625" y1="55.7463125" x2="36.576" y2="59.309" width="2.54" layer="1"/>
+<via x="76.0476" y="95.9612" extent="1-16" drill="0.85"/>
+<via x="76.0222" y="97.9678" extent="1-16" drill="0.85"/>
+<via x="76.0476" y="99.9998" extent="1-16" drill="0.85"/>
 </signal>
 <signal name="R5">
