File: BackPlane.sch (EAGLE design)
At the start: 1 part

Commit message: progress
Parts:
- added U$2, U$3, U$4: THICC_CONNECTOR, THICC_CONNECTOR:THICC_CONNECTOR
Connections:
- new net +12V: U$2.15, U$2.16, U$2.23, U$2.24, U$3.15, U$3.16, U$3.23, U$3.24, U$4.15, U$4.16, U$4.23, U$4.24
- new net +12V_GND: U$2.13, U$2.14, U$2.21, U$2.22, U$3.13, U$3.14, U$3.21, U$3.22, U$4.13, U$4.14, U$4.21, U$4.22
- new net +5V: U$2.11, U$2.12, U$2.19, U$2.20, U$3.11, U$3.12, U$3.19, U$3.20, U$4.11, U$4.12, U$4.19, U$4.20
- new net +5V_GND: U$2.10, U$2.17, U$2.18, U$2.9, U$3.10, U$3.17, U$3.18, U$3.9, U$4.10, U$4.17, U$4.18, U$4.9
- new net B1: U$2.P$13, U$2.P$14, U$2.P$15, U$2.P$16, U$2.P$41, U$2.P$42, U$2.P$43, U$2.P$44, U$4.P$13, U$4.P$14, U$4.P$15, U$4.P$16, U$4.P$41, U$4.P$42, U$4.P$43, U$4.P$44
- new net B2: U$2.P$25, U$2.P$26, U$2.P$27, U$2.P$28, U$2.P$29, U$2.P$30, U$2.P$31, U$2.P$32, U$4.P$25, U$4.P$26, U$4.P$27, U$4.P$28, U$4.P$29, U$4.P$30, U$4.P$31, U$4.P$32
- new net B3: U$2.P$69, U$2.P$70, U$2.P$71, U$2.P$72, U$2.P$77, U$2.P$78, U$2.P$79, U$2.P$80, U$3.P$69, U$3.P$70, U$3.P$71, U$3.P$72, U$3.P$77, U$3.P$78, U$3.P$79, U$3.P$80, U$4.P$69, U$4.P$70, U$4.P$71, U$4.P$72, U$4.P$77, U$4.P$78, U$4.P$79, U$4.P$80
- new net B4: U$2.P$61, U$2.P$62, U$2.P$63, U$2.P$64, U$2.P$81, U$2.P$82, U$2.P$83, U$2.P$84, U$3.P$61, U$3.P$62, U$3.P$63, U$3.P$64, U$3.P$81, U$3.P$82, U$3.P$83, U$3.P$84, U$4.P$61, U$4.P$62, U$4.P$63, U$4.P$64, U$4.P$81, U$4.P$82, U$4.P$83, U$4.P$84
- new net B5: U$3.P$13, U$3.P$14, U$3.P$15, U$3.P$16, U$3.P$41, U$3.P$42, U$3.P$43, U$3.P$44
- new net B6: U$3.P$25, U$3.P$26, U$3.P$27, U$3.P$28, U$3.P$29, U$3.P$30, U$3.P$31, U$3.P$32
- new net CAN_H: U$2.8, U$3.8, U$4.8
- new net CAN_L: U$2.7, U$3.7, U$4.7
- new net R1: U$2.P$1, U$2.P$2, U$2.P$21, U$2.P$22, U$2.P$23, U$2.P$24, U$2.P$3, U$2.P$4, U$4.P$1, U$4.P$2, U$4.P$21, U$4.P$22, U$4.P$23, U$4.P$24, U$4.P$3, U$4.P$4
- new net R2: U$2.P$10, U$2.P$11, U$2.P$12, U$2.P$37, U$2.P$38, U$2.P$39, U$2.P$40, U$2.P$9, U$4.P$10, U$4.P$11, U$4.P$12, U$4.P$37, U$4.P$38, U$4.P$39, U$4.P$40, U$4.P$9
- new net R3: U$2.P$65, U$2.P$66, U$2.P$67, U$2.P$68, U$2.P$85, U$2.P$86, U$2.P$87, U$2.P$88, U$3.P$65, U$3.P$66, U$3.P$67, U$3.P$68, U$4.P$65, U$4.P$66, U$4.P$67, U$4.P$68, U$4.P$85, U$4.P$86, U$4.P$87, U$4.P$88
- new net R4: U$2.P$49, U$2.P$50, U$2.P$51, U$2.P$52, U$2.P$53, U$2.P$54, U$2.P$55, U$2.P$56, U$3.P$49, U$3.P$50, U$3.P$51, U$3.P$52, U$3.P$53, U$3.P$54, U$3.P$55, U$3.P$56, U$4.P$49, U$4.P$50, U$4.P$51, U$4.P$52, U$4.P$53, U$4.P$54, U$4.P$55, U$4.P$56
- new net R5: U$3.P$1, U$3.P$2, U$3.P$21, U$3.P$22, U$3.P$23, U$3.P$24, U$3.P$3, U$3.P$4
- new net R6: U$3.P$10, U$3.P$11, U$3.P$12, U$3.P$37, U$3.P$38, U$3.P$39, U$3.P$40, U$3.P$9
- new net R7: U$3.P$85, U$3.P$86, U$3.P$87, U$3.P$88
- new net Y1: U$2.P$17, U$2.P$18, U$2.P$19, U$2.P$20, U$2.P$45, U$2.P$46, U$2.P$47, U$2.P$48, U$4.P$17, U$4.P$18, U$4.P$19, U$4.P$20, U$4.P$45, U$4.P$46, U$4.P$47, U$4.P$48
- new net Y2: U$2.P$33, U$2.P$34, U$2.P$35, U$2.P$36, U$2.P$5, U$2.P$6, U$2.P$7, U$2.P$8, U$4.P$33, U$4.P$34, U$4.P$35, U$4.P$36, U$4.P$5, U$4.P$6, U$4.P$7, U$4.P$8
- new net Y3: U$2.P$89, U$2.P$90, U$2.P$91, U$2.P$92, U$2.P$93, U$2.P$94, U$2.P$95, U$2.P$96, U$4.P$89, U$4.P$90, U$4.P$91, U$4.P$92, U$4.P$93, U$4.P$94, U$4.P$95, U$4.P$96
- new net Y4: U$2.P$57, U$2.P$58, U$2.P$59, U$2.P$60, U$2.P$73, U$2.P$74, U$2.P$75, U$2.P$76, U$3.P$57, U$3.P$58, U$3.P$59, U$3.P$60, U$3.P$73, U$3.P$74, U$3.P$75, U$3.P$76, U$4.P$57, U$4.P$58, U$4.P$59, U$4.P$60, U$4.P$73, U$4.P$74, U$4.P$75, U$4.P$76
- new net Y5: U$3.P$17, U$3.P$18, U$3.P$19, U$3.P$20, U$3.P$45, U$3.P$46, U$3.P$47, U$3.P$48
- new net Y6: U$3.P$33, U$3.P$34, U$3.P$35, U$3.P$36, U$3.P$5, U$3.P$6, U$3.P$7, U$3.P$8
- new net Y7: U$3.P$89, U$3.P$90, U$3.P$91, U$3.P$92, U$3.P$93, U$3.P$94, U$3.P$95, U$3.P$96

Commit message: names
Connections:
- new net B10: U$4.P$25, U$4.P$26, U$4.P$27, U$4.P$28, U$4.P$29, U$4.P$30, U$4.P$31, U$4.P$32
- new net B11: U$4.P$69, U$4.P$70, U$4.P$71, U$4.P$72, U$4.P$77, U$4.P$78, U$4.P$79, U$4.P$80
- new net B12: U$4.P$61, U$4.P$62, U$4.P$63, U$4.P$64, U$4.P$81, U$4.P$82, U$4.P$83, U$4.P$84
- new net B7: U$3.P$77, U$3.P$78, U$3.P$79, U$3.P$80
- new net B8: U$3.P$61, U$3.P$62, U$3.P$63, U$3.P$64, U$3.P$81, U$3.P$82, U$3.P$83, U$3.P$84
- new net B9: U$4.P$13, U$4.P$14, U$4.P$15, U$4.P$16, U$4.P$41, U$4.P$42, U$4.P$43, U$4.P$44
- new net BY: U$3.P$69, U$3.P$70, U$3.P$71, U$3.P$72
- new net R10: U$4.P$10, U$4.P$11, U$4.P$12, U$4.P$37, U$4.P$38, U$4.P$39, U$4.P$40, U$4.P$9
- new net R11: U$4.P$65, U$4.P$66, U$4.P$67, U$4.P$68, U$4.P$85, U$4.P$86, U$4.P$87, U$4.P$88
- new net R12: U$4.P$49, U$4.P$50, U$4.P$51, U$4.P$52, U$4.P$53, U$4.P$54, U$4.P$55, U$4.P$56
- new net R8: U$3.P$49, U$3.P$50, U$3.P$51, U$3.P$52, U$3.P$53, U$3.P$54, U$3.P$55, U$3.P$56
- new net R9: U$4.P$1, U$4.P$2, U$4.P$21, U$4.P$22, U$4.P$23, U$4.P$24, U$4.P$3, U$4.P$4
- new net Y10: U$4.P$33, U$4.P$34, U$4.P$35, U$4.P$36, U$4.P$5, U$4.P$6, U$4.P$7, U$4.P$8
- new net Y11: U$4.P$89, U$4.P$90, U$4.P$91, U$4.P$92, U$4.P$93, U$4.P$94, U$4.P$95, U$4.P$96
- new net Y12: U$4.P$57, U$4.P$58, U$4.P$59, U$4.P$60, U$4.P$73, U$4.P$74, U$4.P$75, U$4.P$76
- new net Y8: U$3.P$57, U$3.P$58, U$3.P$59, U$3.P$60, U$3.P$73, U$3.P$74, U$3.P$75, U$3.P$76
- new net Y9: U$4.P$17, U$4.P$18, U$4.P$19, U$4.P$20, U$4.P$45, U$4.P$46, U$4.P$47, U$4.P$48
- net B1: no longer U$4.P$13, U$4.P$14, U$4.P$15, U$4.P$16, U$4.P$41, U$4.P$42, U$4.P$43, U$4.P$44
- net B2: no longer U$4.P$25, U$4.P$26, U$4.P$27, U$4.P$28, U$4.P$29, U$4.P$30, U$4.P$31, U$4.P$32
- net B3: no longer U$3.P$69, U$3.P$70, U$3.P$71, U$3.P$72, U$3.P$77, U$3.P$78, U$3.P$79, U$3.P$80, U$4.P$69, U$4.P$70, U$4.P$71, U$4.P$72, U$4.P$77, U$4.P$78, U$4.P$79, U$4.P$80
- net B4: no longer U$3.P$61, U$3.P$62, U$3.P$63, U$3.P$64, U$3.P$81, U$3.P$82, U$3.P$83, U$3.P$84, U$4.P$61, U$4.P$62, U$4.P$63, U$4.P$64, U$4.P$81, U$4.P$82, U$4.P$83, U$4.P$84
- net R1: no longer U$4.P$1, U$4.P$2, U$4.P$21, U$4.P$22, U$4.P$23, U$4.P$24, U$4.P$3, U$4.P$4
- net R2: no longer U$4.P$10, U$4.P$11, U$4.P$12, U$4.P$37, U$4.P$38, U$4.P$39, U$4.P$40, U$4.P$9
- net R3: no longer U$3.P$65, U$3.P$66, U$3.P$67, U$3.P$68, U$4.P$65, U$4.P$66, U$4.P$67, U$4.P$68, U$4.P$85, U$4.P$86, U$4.P$87, U$4.P$88
- net R4: no longer U$3.P$49, U$3.P$50, U$3.P$51, U$3.P$52, U$3.P$53, U$3.P$54, U$3.P$55, U$3.P$56, U$4.P$49, U$4.P$50, U$4.P$51, U$4.P$52, U$4.P$53, U$4.P$54, U$4.P$55, U$4.P$56
- net R7: now also U$3.P$65, U$3.P$66, U$3.P$67, U$3.P$68
- net Y1: no longer U$4.P$17, U$4.P$18, U$4.P$19, U$4.P$20, U$4.P$45, U$4.P$46, U$4.P$47, U$4.P$48
- net Y2: no longer U$4.P$33, U$4.P$34, U$4.P$35, U$4.P$36, U$4.P$5, U$4.P$6, U$4.P$7, U$4.P$8
- net Y3: no longer U$4.P$89, U$4.P$90, U$4.P$91, U$4.P$92, U$4.P$93, U$4.P$94, U$4.P$95, U$4.P$96
- net Y4: no longer U$3.P$57, U$3.P$58, U$3.P$59, U$3.P$60, U$3.P$73, U$3.P$74, U$3.P$75, U$3.P$76, U$4.P$57, U$4.P$58, U$4.P$59, U$4.P$60, U$4.P$73, U$4.P$74, U$4.P$75, U$4.P$76

Commit message: Routing
Connections:
- removed net BY: U$3.P$69, U$3.P$70, U$3.P$71, U$3.P$72
- net +12V: now also U$2.7, U$2.8, U$3.7, U$3.8, U$4.7, U$4.8; no longer U$2.23, U$2.24, U$3.23, U$3.24, U$4.23, U$4.24
- net B7: now also U$3.P$69, U$3.P$70, U$3.P$71, U$3.P$72
- net CAN_H: now also U$2.24, U$3.24, U$4.24; no longer U$2.8, U$3.8, U$4.8
- net CAN_L: now also U$2.23, U$3.23, U$4.23; no longer U$2.7, U$3.7, U$4.7
Changed lines of the file:
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@@
 <net name="CAN_L" class="0">
 <segment>
-<pinref part="U$2" gate="G$1" pin="7"/>
-<wire x1="76.2" y1="170.18" x2="76.2" y2="160.02" width="0.1524" layer="91"/>
-<label x="76.2" y="160.02" size="1.778" layer="95" rot="R90"/>
-</segment>
-<segment>
-<pinref part="U$3" gate="G$1" pin="7"/>
-<wire x1="457.2" y1="182.88" x2="457.2" y2="172.72" width="0.1524" layer="91"/>
-<label x="457.2" y="172.72" size="1.778" layer="95" rot="R90"/>
-</segment>
-<segment>
-<pinref part="U$4" gate="G$1" pin="7"/>
-<wire x1="281.94" y1="-96.52" x2="281.94" y2="-106.68" width="0.1524" layer="91"/>
-<label x="281.94" y="-106.68" size="1.778" layer="95" rot="R90"/>
+<pinref part="U$2" gate="G$1" pin="23"/>
+<wire x1="96.52" y1="208.28" x2="96.52" y2="215.9" width="0.1524" layer="91"/>
+<label x="99.06" y="210.82" size="1.778" layer="95" rot="R90"/>
+</segment>
+<segment>
+<pinref part="U$3" gate="G$1" pin="23"/>
+<wire x1="477.52" y1="220.98" x2="477.52" y2="231.14" width="0.1524" layer="91"/>
+<label x="477.52" y="226.06" size="1.778" layer="95" rot="R90"/>
+</segment>
+<segment>
+<pinref part="U$4" gate="G$1" pin="23"/>
+<wire x1="302.26" y1="-58.42" x2="302.26" y2="-45.72" width="0.1524" layer="91"/>
+<label x="304.8" y="-53.34" size="1.778" layer="95" rot="R90"/>
 </segment>
 </net>
 <net name="CAN_H" class="0">
 <segment>
-<pinref part="U$2" gate="G$1" pin="8"/>
-<wire x1="81.28" y1="170.18" x2="81.28" y2="160.02" width="0.1524" layer="91"/>
-<label x="81.28" y="160.02" size="1.778" layer="95" rot="R90"/>
-</segment>
-<segment>
-<pinref part="U$3" gate="G$1" pin="8"/>
-<wire x1="462.28" y1="182.88" x2="462.28" y2="172.72" width="0.1524" layer="91"/>
-<label x="462.28" y="172.72" size="1.778" layer="95" rot="R90"/>
-</segment>
-<segment>
-<pinref part="U$4" gate="G$1" pin="8"/>
-<wire x1="287.02" y1="-96.52" x2="287.02" y2="-106.68" width="0.1524" layer="91"/>
-<label x="287.02" y="-106.68" size="1.778" layer="95" rot="R90"/>
+<pinref part="U$2" gate="G$1" pin="24"/>
+<wire x1="101.6" y1="208.28" x2="101.6" y2="215.9" width="0.1524" layer="91"/>
+<label x="104.14" y="210.82" size="1.778" layer="95" rot="R90"/>
+</segment>
+<segment>
+<pinref part="U$3" gate="G$1" pin="24"/>
+<wire x1="482.6" y1="220.98" x2="482.6" y2="231.14" width="0.1524" layer="91"/>
+<label x="485.14" y="226.06" size="1.778" layer="95" rot="R90"/>
+</segment>
+<segment>
+<pinref part="U$4" gate="G$1" pin="24"/>
+<wire x1="307.34" y1="-58.42" x2="307.34" y2="-45.72" width="0.1524" layer="91"/>
+<label x="309.88" y="-53.34" size="1.778" layer="95" rot="R90"/>
 </segment>
 </net>
 <net name="+12V" class="0">
-<segment>
-<pinref part="U$2" gate="G$1" pin="23"/>
-<wire x1="96.52" y1="208.28" x2="96.52" y2="213.36" width="0.1524" layer="91"/>
-<wire x1="96.52" y1="213.36" x2="101.6" y2="213.36" width="0.1524" layer="91"/>
-<pinref part="U$2" gate="G$1" pin="24"/>
-<wire x1="101.6" y1="213.36" x2="101.6" y2="208.28" width="0.1524" layer="91"/>
-<wire x1="96.52" y1="213.36" x2="96.52" y2="220.98" width="0.1524" layer="91"/>
-<junction x="96.52" y="213.36"/>
-<label x="96.52" y="215.9" size="1.778" layer="95" rot="R90"/>
-</segment>
 <segment>
 <pinref part="U$2" gate="G$1" pin="16"/>
@@
 </segment>
 <segment>
-<pinref part="U$3" gate="G$1" pin="23"/>
-<wire x1="477.52" y1="220.98" x2="477.52" y2="226.06" width="0.1524" layer="91"/>
-<wire x1="477.52" y1="226.06" x2="482.6" y2="226.06" width="0.1524" layer="91"/>
-<pinref part="U$3" gate="G$1" pin="24"/>
-<wire x1="482.6" y1="226.06" x2="482.6" y2="220.98" width="0.1524" layer="91"/>
-<wire x1="477.52" y1="226.06" x2="477.52" y2="233.68" width="0.1524" layer="91"/>
-<junction x="477.52" y="226.06"/>
-<label x="477.52" y="228.6" size="1.778" layer="95" rot="R90"/>
-</segment>
-<segment>
 <pinref part="U$3" gate="G$1" pin="16"/>
 <wire x1="441.96" y1="220.98" x2="441.96" y2="226.06" width="0.1524" layer="91"/>
@@
 </segment>
 <segment>
-<pinref part="U$4" gate="G$1" pin="23"/>
-<wire x1="302.26" y1="-58.42" x2="302.26" y2="-53.34" width="0.1524" layer="91"/>
-<wire x1="302.26" y1="-53.34" x2="307.34" y2="-53.34" width="0.1524" layer="91"/>
-<pinref part="U$4" gate="G$1" pin="24"/>
-<wire x1="307.34" y1="-53.34" x2="307.34" y2="-58.42" width="0.1524" layer="91"/>
-<wire x1="302.26" y1="-53.34" x2="302.26" y2="-45.72" width="0.1524" layer="91"/>
-<junction x="302.26" y="-53.34"/>
-<label x="302.26" y="-50.8" size="1.778" layer="95" rot="R90"/>
-</segment>
-<segment>
 <pinref part="U$4" gate="G$1" pin="16"/>
 <wire x1="266.7" y1="-58.42" x2="266.7" y2="-53.34" width="0.1524" layer="91"/>
@@
 <junction x="261.62" y="-53.34"/>
 <label x="261.62" y="-50.8" size="1.778" layer="95" rot="R90"/>
+</segment>
+<segment>
+<pinref part="U$2" gate="G$1" pin="8"/>
+<wire x1="81.28" y1="170.18" x2="81.28" y2="162.56" width="0.1524" layer="91"/>
+<pinref part="U$2" gate="G$1" pin="7"/>
+<wire x1="81.28" y1="162.56" x2="76.2" y2="162.56" width="0.1524" layer="91"/>
+<wire x1="76.2" y1="162.56" x2="76.2" y2="170.18" width="0.1524" layer="91"/>
+<wire x1="76.2" y1="162.56" x2="76.2" y2="154.94" width="0.1524" layer="91"/>
+<junction x="76.2" y="162.56"/>
+<label x="76.2" y="154.94" size="1.778" layer="95" rot="R90"/>
+</segment>
+<segment>
+<pinref part="U$3" gate="G$1" pin="7"/>
+<wire x1="457.2" y1="182.88" x2="457.2" y2="180.34" width="0.1524" layer="91"/>
+<wire x1="457.2" y1="180.34" x2="462.28" y2="180.34" width="0.1524" layer="91"/>
+<pinref part="U$3" gate="G$1" pin="8"/>
+<wire x1="462.28" y1="180.34" x2="462.28" y2="182.88" width="0.1524" layer="91"/>
+<wire x1="457.2" y1="180.34" x2="457.2" y2="170.18" width="0.1524" layer="91"/>
+<junction x="457.2" y="180.34"/>
+<label x="457.2" y="170.18" size="1.778" layer="95" rot="R90"/>
+</segment>
+<segment>
+<pinref part="U$4" gate="G$1" pin="7"/>
+<wire x1="281.94" y1="-96.52" x2="281.94" y2="-101.6" width="0.1524" layer="91"/>
+<wire x1="281.94" y1="-101.6" x2="287.02" y2="-101.6" width="0.1524" layer="91"/>
+<pinref part="U$4" gate="G$1" pin="8"/>
+<wire x1="287.02" y1="-101.6" x2="287.02" y2="-96.52" width="0.1524" layer="91"/>
+<wire x1="281.94" y1="-101.6" x2="281.94" y2="-106.68" width="0.1524" layer="91"/>
+<junction x="281.94" y="-101.6"/>
+<label x="284.48" y="-109.22" size="1.778" layer="95" rot="R90"/>
 </segment>
 </net>
@@
 <label x="508" y="124.46" size="1.778" layer="95"/>
 </segment>
+<segment>
+<pinref part="U$3" gate="G$1" pin="P$69"/>
+<wire x1="563.88" y1="111.76" x2="563.88" y2="116.84" width="0.1524" layer="91"/>
+<wire x1="563.88" y1="116.84" x2="558.8" y2="116.84" width="0.1524" layer="91"/>
+<pinref part="U$3" gate="G$1" pin="P$72"/>
+<wire x1="558.8" y1="116.84" x2="553.72" y2="116.84" width="0.1524" layer="91"/>
+<wire x1="553.72" y1="116.84" x2="548.64" y2="116.84" width="0.1524" layer="91"/>
+<wire x1="548.64" y1="116.84" x2="548.64" y2="111.76" width="0.1524" layer="91"/>
+<pinref part="U$3" gate="G$1" pin="P$71"/>
+<wire x1="553.72" y1="111.76" x2="553.72" y2="116.84" width="0.1524" layer="91"/>
+<junction x="553.72" y="116.84"/>
+<pinref part="U$3" gate="G$1" pin="P$70"/>
+<wire x1="558.8" y1="111.76" x2="558.8" y2="116.84" width="0.1524" layer="91"/>
+<junction x="558.8" y="116.84"/>
+<wire x1="548.64" y1="116.84" x2="548.64" y2="124.46" width="0.1524" layer="91"/>
+<junction x="548.64" y="116.84"/>
+<label x="548.64" y="124.46" size="1.778" layer="95"/>
+</segment>
 </net>
 <net name="Y8" class="0">
@@
 </segment>
 </net>
-<net name="BY" class="0">
-<segment>
-<pinref part="U$3" gate="G$1" pin="P$69"/>
-<wire x1="563.88" y1="111.76" x2="563.88" y2="116.84" width="0.1524" layer="91"/>
-<wire x1="563.88" y1="116.84" x2="558.8" y2="116.84" width="0.1524" layer="91"/>
-<pinref part="U$3" gate="G$1" pin="P$72"/>
-<wire x1="558.8" y1="116.84" x2="553.72" y2="116.84" width="0.1524" layer="91"/>
-<wire x1="553.72" y1="116.84" x2="548.64" y2="116.84" width="0.1524" layer="91"/>
-<wire x1="548.64" y1="116.84" x2="548.64" y2="111.76" width="0.1524" layer="91"/>
-<pinref part="U$3" gate="G$1" pin="P$71"/>
-<wire x1="553.72" y1="111.76" x2="553.72" y2="116.84" width="0.1524" layer="91"/>
-<junction x="553.72" y="116.84"/>
-<pinref part="U$3" gate="G$1" pin="P$70"/>
-<wire x1="558.8" y1="111.76" x2="558.8" y2="116.84" width="0.1524" layer="91"/>
-<junction x="558.8" y="116.84"/>
-<wire x1="548.64" y1="116.84" x2="548.64" y2="124.46" width="0.1524" layer="91"/>
-<junction x="548.64" y="116.84"/>
-<label x="548.64" y="124.46" size="1.778" layer="95"/>
-</segment>
-</net>
