File: BackPlane.sch (EAGLE design)
At the start: 4 parts

Commit message: connectors
Parts:
- added ESC5_CON1: 3PINCONNECTOR, afro_20A_esc:3PINCONNECTOR
Changed lines of the file:
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@@
 <layer number="48" name="Document" color="7" fill="1" visible="no" active="no"/>
 <layer number="49" name="Reference" color="7" fill="1" visible="no" active="no"/>
+<layer number="50" name="dxf" color="7" fill="1" visible="no" active="no"/>
 <layer number="51" name="tDocu" color="7" fill="1" visible="no" active="no"/>
 <layer number="52" name="bDocu" color="7" fill="1" visible="no" active="no"/>
+<layer number="53" name="tGND_GNDA" color="7" fill="9" visible="no" active="no"/>
+<layer number="54" name="bGND_GNDA" color="1" fill="9" visible="no" active="no"/>
+<layer number="56" name="wert" color="7" fill="1" visible="no" active="no"/>
+<layer number="57" name="tCAD" color="7" fill="1" visible="no" active="no"/>
+<layer number="59" name="tCarbon" color="7" fill="1" visible="no" active="no"/>
+<layer number="60" name="bCarbon" color="7" fill="1" visible="no" active="no"/>
 <layer number="88" name="SimResults" color="9" fill="1" visible="yes" active="yes"/>
 <layer number="89" name="SimProbes" color="9" fill="1" visible="yes" active="yes"/>
@@
 <layer number="97" name="Info" color="7" fill="1" visible="yes" active="yes"/>
 <layer number="98" name="Guide" color="6" fill="1" visible="yes" active="yes"/>
+<layer number="99" name="SpiceOrder" color="7" fill="1" visible="no" active="no"/>
+<layer number="100" name="Muster" color="7" fill="1" visible="no" active="no"/>
+<layer number="101" name="Patch_Top" color="12" fill="4" visible="yes" active="yes"/>
+<layer number="102" name="Vscore" color="7" fill="1" visible="yes" active="yes"/>
+<layer number="103" name="tMap" color="7" fill="1" visible="yes" active="yes"/>
+<layer number="104" name="Name" color="16" fill="1" visible="yes" active="yes"/>
+<layer number="105" name="tPlate" color="7" fill="1" visible="yes" active="yes"/>
+<layer number="106" name="bPlate" color="7" fill="1" visible="yes" active="yes"/>
+<layer number="107" name="Crop" color="7" fill="1" visible="yes" active="yes"/>
+<layer number="108" name="tplace-old" color="10" fill="1" visible="yes" active="yes"/>
+<layer number="109" name="ref-old" color="11" fill="1" visible="yes" active="yes"/>
+<layer number="110" name="fp0" color="7" fill="1" visible="yes" active="yes"/>
+<layer number="111" name="LPC17xx" color="7" fill="1" visible="yes" active="yes"/>
+<layer number="112" name="tSilk" color="7" fill="1" visible="yes" active="yes"/>
+<layer number="113" name="IDFDebug" color="4" fill="1" visible="yes" active="yes"/>
+<layer number="114" name="Badge_Outline" color="7" fill="1" visible="no" active="yes"/>
+<layer number="115" name="ReferenceISLANDS" color="7" fill="1" visible="no" active="yes"/>
+<layer number="116" name="Patch_BOT" color="9" fill="4" visible="yes" active="yes"/>
+<layer number="118" name="Rect_Pads" color="7" fill="1" visible="no" active="yes"/>
+<layer number="121" name="_tsilk" color="7" fill="1" visible="yes" active="yes"/>
+<layer number="122" name="_bsilk" color="7" fill="1" visible="yes" active="yes"/>
+<layer number="123" name="tTestmark" color="7" fill="1" visible="yes" active="yes"/>
+<layer number="124" name="bTestmark" color="7" fill="1" visible="yes" active="yes"/>
+<layer number="125" name="_tNames" color="7" fill="1" visible="yes" active="yes"/>
+<layer number="126" name="_bNames" color="7" fill="1" visible="yes" active="yes"/>
+<layer number="127" name="_tValues" color="7" fill="1" visible="yes" active="yes"/>
+<layer number="128" name="_bValues" color="7" fill="1" visible="yes" active="yes"/>
+<layer number="129" name="Mask" color="7" fill="1" visible="yes" active="yes"/>
+<layer number="131" name="tAdjust" color="7" fill="1" visible="yes" active="yes"/>
+<layer number="132" name="bAdjust" color="7" fill="1" visible="yes" active="yes"/>
+<layer number="144" name="Drill_legend" color="7" fill="1" visible="yes" active="yes"/>
+<layer number="150" name="Notes" color="7" fill="1" visible="yes" active="yes"/>
+<layer number="151" name="HeatSink" color="7" fill="1" visible="yes" active="yes"/>
+<layer number="152" name="_bDocu" color="7" fill="1" visible="yes" active="yes"/>
+<layer number="153" name="FabDoc1" color="7" fill="1" visible="yes" active="yes"/>
+<layer number="154" name="FabDoc2" color="7" fill="1" visible="yes" active="yes"/>
+<layer number="155" name="FabDoc3" color="7" fill="1" visible="yes" active="yes"/>
+<layer number="199" name="Contour" color="7" fill="1" visible="yes" active="yes"/>
+<layer number="200" name="200bmp" color="1" fill="10" visible="yes" active="yes"/>
+<layer number="201" name="201bmp" color="2" fill="10" visible="yes" active="yes"/>
+<layer number="202" name="202bmp" color="3" fill="10" visible="yes" active="yes"/>
+<layer number="203" name="203bmp" color="4" fill="10" visible="yes" active="yes"/>
+<layer number="204" name="204bmp" color="5" fill="10" visible="yes" active="yes"/>
+<layer number="205" name="205bmp" color="6" fill="10" visible="yes" active="yes"/>
+<layer number="206" name="206bmp" color="7" fill="10" visible="yes" active="yes"/>
+<layer number="207" name="207bmp" color="8" fill="10" visible="yes" active="yes"/>
+<layer number="208" name="208bmp" color="9" fill="10" visible="yes" active="yes"/>
+<layer number="209" name="209bmp" color="7" fill="1" visible="yes" active="yes"/>
+<layer number="210" name="210bmp" color="7" fill="1" visible="yes" active="yes"/>
+<layer number="211" name="211bmp" color="7" fill="1" visible="yes" active="yes"/>
+<layer number="212" name="212bmp" color="7" fill="1" visible="yes" active="yes"/>
+<layer number="213" name="213bmp" color="7" fill="1" visible="yes" active="yes"/>
+<layer number="214" name="214bmp" color="7" fill="1" visible="yes" active="yes"/>
+<layer number="215" name="215bmp" color="7" fill="1" visible="yes" active="yes"/>
+<layer number="216" name="216bmp" color="7" fill="1" visible="yes" active="yes"/>
+<layer number="217" name="217bmp" color="18" fill="1" visible="no" active="no"/>
+<layer number="218" name="218bmp" color="19" fill="1" visible="no" active="no"/>
+<layer number="219" name="219bmp" color="20" fill="1" visible="no" active="no"/>
+<layer number="220" name="220bmp" color="21" fill="1" visible="no" active="no"/>
+<layer number="221" name="221bmp" color="22" fill="1" visible="no" active="no"/>
+<layer number="222" name="222bmp" color="23" fill="1" visible="no" active="no"/>
+<layer number="223" name="223bmp" color="24" fill="1" visible="no" active="no"/>
+<layer number="224" name="224bmp" color="25" fill="1" visible="no" active="no"/>
+<layer number="225" name="225bmp" color="7" fill="1" visible="yes" active="yes"/>
+<layer number="226" name="226bmp" color="7" fill="1" visible="yes" active="yes"/>
+<layer number="227" name="227bmp" color="7" fill="1" visible="yes" active="yes"/>
+<layer number="228" name="228bmp" color="7" fill="1" visible="yes" active="yes"/>
+<layer number="229" name="229bmp" color="7" fill="1" visible="yes" active="yes"/>
+<layer number="230" name="230bmp" color="7" fill="1" visible="yes" active="yes"/>
+<layer number="231" name="231bmp" color="7" fill="1" visible="yes" active="yes"/>
+<layer number="232" name="Eagle3D_PG2" color="7" fill="1" visible="yes" active="yes"/>
+<layer number="233" name="Eagle3D_PG3" color="7" fill="1" visible="yes" active="yes"/>
+<layer number="248" name="Housing" color="7" fill="1" visible="yes" active="yes"/>
+<layer number="249" name="Edge" color="7" fill="1" visible="yes" active="yes"/>
+<layer number="250" name="Descript" color="3" fill="1" visible="no" active="no"/>
+<layer number="251" name="SMDround" color="12" fill="11" visible="no" active="no"/>
+<layer number="254" name="cooling" color="7" fill="1" visible="yes" active="yes"/>
+<layer number="255" name="routoute" color="7" fill="1" visible="yes" active="yes"/>
 </layers>
 <schematic xreflabel="%F%N/%S.%C%R" xrefpart="/%S.%C%R">
@@
 <part name="U$3" library="THICC_CONNECTOR" deviceset="THICC_CONNECTOR" device=""/>
 <part name="U$4" library="THICC_CONNECTOR" deviceset="THICC_CONNECTOR" device=""/>
+<part name="ESC5_CON1" library="afro_20A_esc" deviceset="3PINCONNECTOR" device=""/>
 </parts>
 <sheets>
@@
 <instance part="U$3" gate="G$1" x="454.66" y="91.44" rot="R90"/>
 <instance part="U$4" gate="G$1" x="279.4" y="-187.96" rot="R90"/>
+<instance part="ESC5_CON1" gate="G$1" x="185.42" y="238.76" rot="R90">
+<attribute name="NAME" x="177.8" y="231.14" size="1.778" layer="95" rot="R90"/>
+</instance>
 </instances>
 <busses>

Commit message: routing
Parts:
- added ESC5_CON10, ESC5_CON11, ESC5_CON12, ESC5_CON2, ESC5_CON3, ESC5_CON4, ESC5_CON5, ESC5_CON6, ESC5_CON7, ESC5_CON8, ESC5_CON9: 3PINCONNECTOR, afro_20A_esc:3PINCONNECTOR
Connections:
- net B1: now also ESC5_CON1.C
- net B10: now also ESC5_CON10.C
- net B11: now also ESC5_CON11.C
- net B12: now also ESC5_CON12.C
- net B2: now also ESC5_CON2.C
- net B3: now also ESC5_CON3.C
- net B4: now also ESC5_CON4.C
- net B5: now also ESC5_CON5.C
- net B6: now also ESC5_CON6.C
- net B7: now also ESC5_CON7.C
- net B8: now also ESC5_CON8.C
- net B9: now also ESC5_CON9.C
- net R1: now also ESC5_CON1.A
- net R10: now also ESC5_CON10.A
- net R11: now also ESC5_CON11.A
- net R12: now also ESC5_CON12.A
- net R2: now also ESC5_CON2.A
- net R3: now also ESC5_CON3.A
- net R4: now also ESC5_CON4.A
- net R5: now also ESC5_CON5.A
- net R6: now also ESC5_CON6.A
- net R7: now also ESC5_CON7.A
- net R8: now also ESC5_CON8.A
- net R9: now also ESC5_CON9.A
- net Y1: now also ESC5_CON1.B
- net Y10: now also ESC5_CON10.B
- net Y11: now also ESC5_CON11.B
- net Y12: now also ESC5_CON12.B
- net Y2: now also ESC5_CON2.B
- net Y3: now also ESC5_CON3.B
- net Y4: now also ESC5_CON4.B
- net Y5: now also ESC5_CON5.B
- net Y6: now also ESC5_CON6.B
- net Y7: now also ESC5_CON7.B
- net Y8: now also ESC5_CON8.B
- net Y9: now also ESC5_CON9.B

Commit message: More Routing
Parts:
- added U$10, U$5, U$6: T2I, BackplaneParts:T2I
Connections:
- net +5V: now also U$5.2, U$5.3, U$5.4
- net +5V_GND: now also U$6.2, U$6.3, U$6.4
- net CAN_H: now also U$10.2
- net CAN_L: now also U$10.3
Changed lines of the file:
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@@
 <part name="ESC5_CON11" library="afro_20A_esc" deviceset="3PINCONNECTOR" device=""/>
 <part name="ESC5_CON12" library="afro_20A_esc" deviceset="3PINCONNECTOR" device=""/>
+<part name="U$10" library="BackplaneParts" deviceset="T2I" device=""/>
+<part name="U$5" library="BackplaneParts" deviceset="T2I" device=""/>
+<part name="U$6" library="BackplaneParts" deviceset="T2I" device=""/>
 </parts>
 <sheets>
@@
 <attribute name="NAME" x="447.04" y="-53.34" size="1.778" layer="95" rot="R90"/>
 </instance>
+<instance part="U$10" gate="G$1" x="294.64" y="236.22" rot="R270"/>
+<instance part="U$5" gate="G$1" x="294.64" y="213.36" rot="R270"/>
+<instance part="U$6" gate="G$1" x="294.64" y="193.04" rot="R270"/>
 </instances>
 <busses>
@@
 <label x="304.8" y="-53.34" size="1.778" layer="95" rot="R90"/>
 </segment>
+<segment>
+<pinref part="U$10" gate="G$1" pin="3"/>
+<wire x1="307.34" y1="228.6" x2="314.96" y2="228.6" width="0.1524" layer="91"/>
+<label x="309.88" y="228.6" size="1.778" layer="95"/>
+</segment>
 </net>
 <net name="CAN_H" class="0">
@@
 <wire x1="307.34" y1="-58.42" x2="307.34" y2="-45.72" width="0.1524" layer="91"/>
 <label x="309.88" y="-53.34" size="1.778" layer="95" rot="R90"/>
+</segment>
+<segment>
+<pinref part="U$10" gate="G$1" pin="2"/>
+<wire x1="307.34" y1="231.14" x2="314.96" y2="231.14" width="0.1524" layer="91"/>
+<label x="309.88" y="231.14" size="1.778" layer="95"/>
 </segment>
 </net>
@@
 <label x="302.26" y="-106.68" size="1.778" layer="95" rot="R90"/>
 </segment>
+<segment>
+<pinref part="U$5" gate="G$1" pin="4"/>
+<wire x1="307.34" y1="203.2" x2="314.96" y2="203.2" width="0.1524" layer="91"/>
+<wire x1="314.96" y1="203.2" x2="314.96" y2="205.74" width="0.1524" layer="91"/>
+<pinref part="U$5" gate="G$1" pin="3"/>
+<wire x1="314.96" y1="205.74" x2="307.34" y2="205.74" width="0.1524" layer="91"/>
+<pinref part="U$5" gate="G$1" pin="2"/>
+<wire x1="314.96" y1="205.74" x2="314.96" y2="208.28" width="0.1524" layer="91"/>
+<wire x1="314.96" y1="208.28" x2="307.34" y2="208.28" width="0.1524" layer="91"/>
+<junction x="314.96" y="205.74"/>
+<wire x1="314.96" y1="203.2" x2="320.04" y2="203.2" width="0.1524" layer="91"/>
+<junction x="314.96" y="203.2"/>
+<label x="317.5" y="203.2" size="1.778" layer="95"/>
+</segment>
 </net>
 <net name="+5V_GND" class="0">
@@
 <label x="292.1" y="-111.76" size="1.778" layer="95" rot="R90"/>
 </segment>
-</net>
+<segment>
+<pinref part="U$6" gate="G$1" pin="4"/>
+<wire x1="307.34" y1="182.88" x2="314.96" y2="182.88" width="0.1524" layer="91"/>
+<wire x1="314.96" y1="182.88" x2="314.96" y2="185.42" width="0.1524" layer="91"/>
+<pinref part="U$6" gate="G$1" pin="3"/>
+<wire x1="314.96" y1="185.42" x2="307.34" y2="185.42" width="0.1524" layer="91"/>
+<pinref part="U$6" gate="G$1" pin="2"/>
+<wire x1="314.96" y1="185.42" x2="314.96" y2="187.96" width="0.1524" layer="91"/>
+<wire x1="314.96" y1="187.96" x2="307.34" y2="187.96" width="0.1524" layer="91"/>
+<junction x="314.96" y="185.42"/>
+<wire x1="314.96" y1="182.88" x2="320.04" y2="182.88" width="0.1524" layer="91"/>
+<junction x="314.96" y="182.88"/>
+<label x="317.5" y="182.88" size="1.778" layer="95"/>
+</segment>
+</net>

Commit message: Routed
Parts:
- added U$11, U$12, U$15, U$16, U$7, U$8, U$9: T2I, BackplaneParts:T2I
Connections:
- net +12V: now also U$15.2, U$15.3, U$15.4, U$7.2, U$7.3, U$7.4, U$9.2, U$9.3, U$9.4
- net +12V_GND: now also U$11.2, U$11.3, U$11.4, U$16.2, U$16.3, U$16.4, U$2.5, U$2.6, U$3.5, U$3.6, U$4.5, U$4.6, U$8.2, U$8.3, U$8.4; no longer U$2.21, U$2.22, U$3.21, U$3.22, U$4.21, U$4.22
- net +5V: now also U$2.3, U$2.4, U$3.3, U$3.4, U$4.3, U$4.4; no longer U$2.19, U$2.20, U$3.19, U$3.20, U$4.19, U$4.20
- net +5V_GND: now also U$2.1, U$2.2, U$3.1, U$3.2, U$4.1, U$4.2; no longer U$2.17, U$2.18, U$3.17, U$3.18, U$4.17, U$4.18
- net CAN_H: now also U$12.2
- net CAN_L: now also U$12.3
Other:
- note added: "12V to Logic"
- note added: "12V to Solenoid Box"
- note added: "5V to Logic"
- note added: "Add Holes for EXTRA CAN HL AND 12/5 Volts"
- note added: "CAN to Logic"

Commit message: final stuff
Other:
- note removed: "Add Holes for EXTRA CAN HL AND 12/5 Volts"
Changed lines of the file:
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@@
 <text x="304.8" y="213.36" size="1.778" layer="91">5V to Logic</text>
 <text x="302.26" y="243.84" size="1.778" layer="91">CAN to Logic</text>
-<text x="325.12" y="81.28" size="1.778" layer="91">Add Holes for EXTRA CAN HL AND 12/5 Volts</text>
 </plain>
 <instances>
